Commit message: modify the robot

File: tennis_bot_description/src/description/tennis_bot_description.urdf (robot description, URDF)
Before this commit: robot tennis_bot, 2 links, 1 joints
Links:
- added link base_top_link; collision box size=0.38 0.27 0.02; visual box size=0.38 0.27 0.02
Joints:
- added joint base_top_joint: type fixed, parent base_link, child base_top_link, origin xyz=0.0 0.0 0.08 rpy=0 0 0

Commit message: changement de dimensions du robot

File: tennis_bot_description/src/description/tennis_bot_description.urdf (robot description, URDF)
Before this commit: robot tennis_bot, 4 links, 3 joints
Links:
- link base_top_link_green: geometry collision box size=${(base_length-0.04)/2} ${base_width-0.04} 0.02; visual box size=${(base_length-0.04)/2} ${base_width-0.04} 0.02
- link base_top_link_red: geometry collision box size=${(base_length-0.04)/2} ${base_width-0.04} 0.02; visual box size=${(base_length-0.04)/2} ${base_width-0.04} 0.02
Joints:
- joint base_top_joint_green: origin xyz=-0.095 0.0 0.08 rpy=0 0 0 -> xyz=${-(base_length-0.04)/4} 0.0 ${base_height/2} rpy=0 0 0
- joint base_top_joint_red: origin xyz=0.095 0.0 0.08 rpy=0 0 0 -> xyz=${(base_length-0.04)/4} 0.0 ${base_height/2} rpy=0 0 0
